Commit message: Addes a launcher with inertias and fixed bugs regarding subscriber in the gui

File: phantomx_pincher/urdf/phantomx_description_inercias.xacro (robot description, xacro)
@@ -2,5 +2,5 @@
 <robot name="phantomx_pincher" xmlns:xacro="http://ros.org/wiki/xacro">
 <!-- -|-|-|-|-|-|-|-|- INCLUDE -|-|-|-|-|-|-|-|- -->
-<xacro:include filename="$(find phantomx_pincher)/urdf/phantomx_parameters.xacro" />
+<xacro:include filename="$(find phantomx_pincher)/urdf/phantomx_parameters_inercias.xacro" />
 <!-- -|-|-|-|-|-|-|-|- ROBOT DESCRIPTION -|-|-|-|-|-|-|-|- -->
 <!-- Gazebo World link -->
@@ -128,5 +128,5 @@
     origin_xyz="${l4} 0 -${offset_finger}"
     axis_xyz="0 0 1"
-    limit_e="10" limit_l="0" limit_u="${joint_gripper_limit}" limit_v="0.01"
+    limit_e="100" limit_l="0" limit_u="${joint_gripper_limit}" limit_v="0.01"
 />
 <!-- Joint-Servomotor-Gripper 2 -->
@@ -139,5 +139,5 @@
     origin_xyz="${l4} 0 ${offset_finger}"
     axis_xyz="0 0 1"
-    limit_e="10" limit_l="0" limit_u="${joint_gripper_limit}" limit_v="0.01"
+    limit_e="100" limit_l="0" limit_u="${joint_gripper_limit}" limit_v="0.01"
 />
 <!-- Link-Gripper Finger 1 -->
@@ -187,24 +187,24 @@
 />
 <!-- Joint-Fixed-Camera-->
-<!--<joint_camera-->
-<!--    name="joint_camera_1" -->
-<!--    type="fixed"-->
-<!--    parent="world"-->
-<!--    child="link_fixed_camera"-->
-<!--    origin_rpy="0 0 ${8*M_PI/6}" -->
-<!--    origin_xyz="0.4 0.4 0"-->
-<!--    axis_xyz="1 0 0" -->
-<!--/>-->
+<joint_camera
+    name="joint_camera_1"
+    type="fixed"
+    parent="world"
+    child="link_fixed_camera"
+    origin_rpy="0 0 ${8*M_PI/6}"
+    origin_xyz="0.4 0.4 0"
+    axis_xyz="1 0 0"
+/>
 <!-- Link-Fixed-Camera-->
-<!--<link_camera-->
-<!--    name="link_fixed_camera"-->
-<!--    origin_rpy="0 0 0" -->
-<!--    origin_xyz="0 0 0"-->
-<!--    inertial_rpy="0 0 0" -->
-<!--    inertial_xyz="${camera_size/2} 0 0"-->
-<!--    mass="${camera_mass}"-->
-<!--    ixx="${camera_ixx}" ixy="${camera_ixy}" ixz="${camera_ixz}"-->
-<!--    iyy="${camera_iyy}" iyz="${camera_iyz}" izz="${camera_izz}"-->
-<!--/> -->
+<link_camera
+    name="link_fixed_camera"
+    origin_rpy="0 0 0"
+    origin_xyz="0 0 0"
+    inertial_rpy="0 0 0"
+    inertial_xyz="${camera_size/2} 0 0"
+    mass="${camera_mass}"
+    ixx="${camera_ixx}" ixy="${camera_ixy}" ixz="${camera_ixz}"
+    iyy="${camera_iyy}" iyz="${camera_iyz}" izz="${camera_izz}"
+/>
 <!-- -|-|-|-|-|-|-|-|- GAZEBO PLUGIN -|-|-|-|-|-|-|-|- -->
 <gazebo>
@@ -212,19 +212,19 @@
         <robotNamespace>/phantomx_pincher</robotNamespace>
     </plugin>
-    <plugin name="gazebo_grasp_fix" filename="libgazebo_grasp_fix.so">
-        <arm>
-           <arm_name>arm_pincher</arm_name>
-           <palm_link>link_4</palm_link>
-           <gripper_link>link_finger_1</gripper_link>
-           <gripper_link>link_finger_1</gripper_link>
-        </arm>
-       <forces_angle_tolerance>100</forces_angle_tolerance>
-       <update_rate>100</update_rate>
-       <grip_count_threshold>5</grip_count_threshold>
-       <max_grip_count>10</max_grip_count>
-       <release_tolerance>0.005</release_tolerance>
-       <disable_collisions_on_attach>true</disable_collisions_on_attach>
-       <contact_topic>__default_topic__</contact_topic>
-    </plugin>
+<!--    <plugin name="gazebo_grasp_fix" filename="libgazebo_grasp_fix.so">-->
+<!--        <arm>-->
+<!--           <arm_name>phantomx_pincher</arm_name>-->
+<!--           <palm_link>link_4</palm_link>-->
+<!--           <gripper_link>link_finger_1</gripper_link>-->
+<!--           <gripper_link>link_finger_1</gripper_link>-->
+<!--        </arm>-->
+<!--       <forces_angle_tolerance>100</forces_angle_tolerance>-->
+<!--       <update_rate>5</update_rate>-->
+<!--       <grip_count_threshold>4</grip_count_threshold>-->
+<!--       <max_grip_count>8</max_grip_count>-->
+<!--       <release_tolerance>0.005</release_tolerance>-->
+<!--       <disable_collisions_on_attach>false</disable_collisions_on_attach>-->
+<!--       <contact_topic>__default_topic__</contact_topic>-->
+<!--    </plugin>-->
 </gazebo>
 <gazebo reference="link_gripper_camera">
@@ -264,39 +264,39 @@
 </sensor>
 </gazebo>
-<!--<gazebo reference="link_fixed_camera">-->
-<!--<sensor type="camera" name="camera_1">-->
-<!--  <update_rate>5</update_rate>-->
-<!--  <camera name="head">-->
-<!--    <horizontal_fov>1.3962634</horizontal_fov>-->
-<!--    <image>-->
-<!--      <width>800</width>-->
-<!--      <height>800</height>-->
-<!--      <format>R8G8B8</format>-->
-<!--    </image>-->
-<!--    <clip>-->
-<!--      <near>0.02</near>-->
-<!--      <far>300</far>-->
-<!--    </clip>-->
-<!--    <noise>-->
-<!--      <type>gaussian</type>-->
-<!--      <mean>0.0</mean>-->
-<!--      <stddev>0.007</stddev>-->
-<!--    </noise>-->
-<!--  </camera>-->
-<!--  <plugin name="camera_controller" filename="libgazebo_ros_camera.so">-->
-<!--    <alwaysOn>true</alwaysOn>-->
-<!--    <updateRate>0.0</updateRate>-->
-<!--    <cameraName>camera_1</cameraName>-->
-<!--    <imageTopicName>image_raw</imageTopicName>-->
-<!--    <cameraInfoTopicName>camera_info</cameraInfoTopicName>-->
-<!--    <frameName>camera_link</frameName>-->
-<!--    <hackBaseline>0.07</hackBaseline>-->
-<!--    <distortionK1>0.0</distortionK1>-->
-<!--    <distortionK2>0.0</distortionK2>-->
-<!--    <distortionK3>0.0</distortionK3>-->
-<!--    <distortionT1>0.0</distortionT1>-->
-<!--    <distortionT2>0.0</distortionT2>-->
-<!--  </plugin>-->
-<!--</sensor>-->
-<!--</gazebo>-->
+<gazebo reference="link_fixed_camera">
+<sensor type="camera" name="camera_1">
+  <update_rate>5</update_rate>
+  <camera name="head">
+    <horizontal_fov>1.3962634</horizontal_fov>
+    <image>
+      <width>800</width>
+      <height>800</height>
+      <format>R8G8B8</format>
+    </image>
+    <clip>
+      <near>0.02</near>
+      <far>300</far>
+    </clip>
+    <noise>
+      <type>gaussian</type>
+      <mean>0.0</mean>
+      <stddev>0.007</stddev>
+    </noise>
+  </camera>
+  <plugin name="camera_controller" filename="libgazebo_ros_camera.so">
+    <alwaysOn>true</alwaysOn>
+    <updateRate>0.0</updateRate>
+    <cameraName>camera_1</cameraName>
+    <imageTopicName>image_raw</imageTopicName>
+    <cameraInfoTopicName>camera_info</cameraInfoTopicName>
+    <frameName>camera_link</frameName>
+    <hackBaseline>0.07</hackBaseline>
+    <distortionK1>0.0</distortionK1>
+    <distortionK2>0.0</distortionK2>
+    <distortionK3>0.0</distortionK3>
+    <distortionT1>0.0</distortionT1>
+    <distortionT2>0.0</distortionT2>
+  </plugin>
+</sensor>
+</gazebo>
 </robot>

File: phantomx_pincher/urdf/phantomx_parameters_inercias.xacro (robot description, xacro)
@@ -18,52 +18,52 @@
 </material>
 <!-- Mass and Inertia -->
-<xacro:property name="link_base_mass" value="0.33520"/>
-<xacro:property name="link_base_ixx" value="0.0"/>
-<xacro:property name="link_base_ixy" value="0.0"/>
-<xacro:property name="link_base_ixz" value="0.0"/>
-<xacro:property name="link_base_iyy" value="0.0"/>
-<xacro:property name="link_base_iyz" value="0.0"/>
-<xacro:property name="link_base_izz" value="0.0"/>
-<xacro:property name="link_1_mass" value="0.11748"/>
-<xacro:property name="link_1_ixx" value="0.0"/>
-<xacro:property name="link_1_ixy" value="0.0"/>
-<xacro:property name="link_1_ixz" value="0.0"/>
-<xacro:property name="link_1_iyy" value="0.0"/>
-<xacro:property name="link_1_iyz" value="0.0"/>
-<xacro:property name="link_1_izz" value="0.0"/>
-<xacro:property name="link_2_mass" value="0.16239"/>
-<xacro:property name="link_2_ixx" value="0.0"/>
-<xacro:property name="link_2_ixy" value="0.0"/>
-<xacro:property name="link_2_ixz" value="0.0"/>
-<xacro:property name="link_2_iyy" value="0.0"/>
-<xacro:property name="link_2_iyz" value="0.0"/>
-<xacro:property name="link_2_izz" value="0.0"/>
-<xacro:property name="link_3_mass" value="0.16239"/>
-<xacro:property name="link_3_ixx" value="0.0"/>
-<xacro:property name="link_3_ixy" value="0.0"/>
-<xacro:property name="link_3_ixz" value="0.0"/>
-<xacro:property name="link_3_iyy" value="0.0"/>
-<xacro:property name="link_3_iyz" value="0.0"/>
-<xacro:property name="link_3_izz" value="0.0"/>
-<xacro:property name="link_4_mass" value="0.16012"/>
-<xacro:property name="link_4_ixx" value="0.0"/>
-<xacro:property name="link_4_ixy" value="0.0"/>
-<xacro:property name="link_4_ixz" value="0.0"/>
-<xacro:property name="link_4_iyy" value="0.0"/>
-<xacro:property name="link_4_iyz" value="0.0"/>
-<xacro:property name="link_4_izz" value="0.0"/>
-<xacro:property name="finger_mass" value="0.01769"/>
-<xacro:property name="finger_ixx" value="0.0"/>
-<xacro:property name="finger_ixy" value="0.0"/>
-<xacro:property name="finger_ixz" value="0.0"/>
-<xacro:property name="finger_iyy" value="0.0"/>
-<xacro:property name="finger_iyz" value="0.0"/>
-<xacro:property name="finger_izz" value="0.0"/>
+<xacro:property name="link_base_mass" value="0.131541100"/>
+<xacro:property name="link_base_ixx" value="0.000212112"/>
+<xacro:property name="link_base_ixy" value="0.000000038"/>
+<xacro:property name="link_base_ixz" value="-0.000051900"/>
+<xacro:property name="link_base_iyy" value="0.000291337"/>
+<xacro:property name="link_base_iyz" value="-0.000000054"/>
+<xacro:property name="link_base_izz" value="0.000276625"/>
+<xacro:property name="link_1_mass" value="0.046266180"/>
+<xacro:property name="link_1_ixx" value="0.000014303"/>
+<xacro:property name="link_1_ixy" value="-0.000000001"/>
+<xacro:property name="link_1_ixz" value="0.000000010"/>
+<xacro:property name="link_1_iyy" value="0.000012129"/>
+<xacro:property name="link_1_iyz" value="-0.000000150"/>
+<xacro:property name="link_1_izz" value="0.000007453"/>
+<xacro:property name="link_2_mass" value="0.063502600"/>
+<xacro:property name="link_2_ixx" value="0.000048752"/>
+<xacro:property name="link_2_ixy" value="-0.000000001"/>
+<xacro:property name="link_2_ixz" value="-0.000000008"/>
+<xacro:property name="link_2_iyy" value="0.000043805"/>
+<xacro:property name="link_2_iyz" value="-0.000000528"/>
+<xacro:property name="link_2_izz" value="0.000012251"/>
+<xacro:property name="link_3_mass" value="0.063502600"/>
+<xacro:property name="link_3_ixx" value="0.000048752"/>
+<xacro:property name="link_3_ixy" value="-0.000000001"/>
+<xacro:property name="link_3_ixz" value="-0.000000008"/>
+<xacro:property name="link_3_iyy" value="0.000043805"/>
+<xacro:property name="link_3_iyz" value="-0.000000528"/>
+<xacro:property name="link_3_izz" value="0.000012251"/>
+<xacro:property name="link_4_mass" value="0.063049010"/>
+<xacro:property name="link_4_ixx" value="0.000022624"/>
+<xacro:property name="link_4_ixy" value="0.000000016"/>
+<xacro:property name="link_4_ixz" value="0.000000924"/>
+<xacro:property name="link_4_iyy" value="0.000027037"/>
+<xacro:property name="link_4_iyz" value="-0.000000005"/>
+<xacro:property name="link_4_izz" value="0.000021160"/>
+<xacro:property name="finger_mass" value="0.006803850"/>
+<xacro:property name="finger_ixx" value="0.000001127"/>
+<xacro:property name="finger_ixy" value="0.000000000"/>
+<xacro:property name="finger_ixz" value="0.000000000"/>
+<xacro:property name="finger_iyy" value="0.000001776"/>
+<xacro:property name="finger_iyz" value="-0.000000278"/>
+<xacro:property name="finger_izz" value="0.000001162"/>
 <!-- Joint-Servomotor Position Limits -150,150 deg -->
 <xacro:property name="joint_lower" value="-2.61799" />
 <xacro:property name="joint_upper" value="2.61799" />
 <!-- Joint-Servomotor Effort-Velocity Limits -->
-<xacro:property name="le" value="100" />
-<xacro:property name="lv" value="0.5" />
+<xacro:property name="le" value="5" />
+<xacro:property name="lv" value="5" />
 <!-- Gripper Joint limits  -->
 <xacro:property name="joint_gripper_limit" value="0.02" />
@@ -173,7 +173,7 @@
         </visual>
         <inertial>
-            <mass value="0" />
+            <mass value="${mass}" />
             <origin rpy="${inertial_rpy}" xyz="${inertial_xyz}" />
-            <inertia ixx="0" ixy="0" ixz="0" iyy="0" iyz="0" izz="0" />
+            <inertia ixx="${ixx}" ixy="${ixy}" ixz="${ixz}" iyy="${iyy}" iyz="${iyz}" izz="${izz}" />
         </inertial>
     </link>
