Commit message: Reorganizar los archivos para mayor claridad y actualizarlos a las versiones màs recientes
Se creò una carpeta llamada documentos, que contiene los documentos pertienentes, tambièn se creo un acarpeta de imàgenes con las imàgenes necesarias, se creo un acarpeta de paquetes de ros donde se guardaron todos los paquetes necesarios, no solo el dle phantom. Tambièn se actualizaron los archivos de la GUI y se borraron los archivos antiguos de la GUI

File: Packages/phantomx_pincher/urdf/phantomx_description.xacro (robot description, xacro)
@@ -128,5 +128,5 @@
     origin_xyz="${l4} 0 -${offset_finger}"
     axis_xyz="0 0 1"
-    limit_e="10" limit_l="0" limit_u="${joint_gripper_limit}" limit_v="0.01"
+    limit_e="10" limit_l="0" limit_u="${joint_gripper_limit}" limit_v="0.001"
 />
 <!-- Joint-Servomotor-Gripper 2 -->
@@ -139,30 +139,70 @@
     origin_xyz="${l4} 0 ${offset_finger}"
     axis_xyz="0 0 1"
-    limit_e="10" limit_l="0" limit_u="${joint_gripper_limit}" limit_v="0.01"
+    limit_e="10" limit_l="0" limit_u="${joint_gripper_limit}" limit_v="0.001"
 />
 <!-- Link-Gripper Finger 1 -->
-<link_phantomx
-    name="link_finger_1"
-    origin_rpy="${M_PI/2} 0 ${M_PI/2}"
-    origin_xyz="-0.019 0 0"
-    inertial_rpy="${M_PI/2} 0 ${M_PI/2}"
-    inertial_xyz="0.006186000 0 0.011269000"
-    meshfile="package://phantomx_pincher/meshes/finger.dae"
-    mass="${finger_mass}"
-    ixx="${finger_ixx}" ixy="${finger_ixy}" ixz="${finger_ixz}"
-    iyy="${finger_iyy}" iyz="${finger_iyz}" izz="${finger_izz}"
-/>
+<!--<link_phantomx-->
+<!--    name="link_finger_1"-->
+<!--    origin_rpy="${M_PI/2} 0 ${M_PI/2}" -->
+<!--    origin_xyz="-0.019 0 0"-->
+<!--    inertial_rpy="${M_PI/2} 0 ${M_PI/2}" -->
+<!--    inertial_xyz="0.006186000 0 0.011269000"-->
+<!--    meshfile="package://phantomx_pincher/meshes/finger.dae"-->
+<!--    mass="${finger_mass}"-->
+<!--    ixx="${finger_ixx}" ixy="${finger_ixy}" ixz="${finger_ixz}"-->
+<!--    iyy="${finger_iyy}" iyz="${finger_iyz}" izz="${finger_izz}"	-->
+<!--/> -->
 <!-- Link-Gripper Finger 2 -->
-<link_phantomx
-    name="link_finger_2"
-    origin_rpy="${M_PI/2} 0 ${M_PI/2}"
-    origin_xyz="-0.019 0 0"
-    inertial_rpy="${M_PI/2} 0 ${M_PI/2}"
-    inertial_xyz="0.006186000 0 0.011269000"
-    meshfile="package://phantomx_pincher/meshes/finger.dae"
-    mass="${finger_mass}"
-    ixx="${finger_ixx}" ixy="${finger_ixy}" ixz="${finger_ixz}"
-    iyy="${finger_iyy}" iyz="${finger_iyz}" izz="${finger_izz}"
-/>
+<!--<link_phantomx-->
+<!--    name="link_finger_2"-->
+<!--    origin_rpy="${M_PI/2} 0 ${M_PI/2}" -->
+<!--    origin_xyz="-0.019 0 0"-->
+<!--    inertial_rpy="${M_PI/2} 0 ${M_PI/2}" -->
+<!--    inertial_xyz="0.006186000 0 0.011269000"-->
+<!--    meshfile="package://phantomx_pincher/meshes/finger.dae"-->
+<!--    mass="${finger_mass}"-->
+<!--    ixx="${finger_ixx}" ixy="${finger_ixy}" ixz="${finger_ixz}"-->
+<!--    iyy="${finger_iyy}" iyz="${finger_iyz}" izz="${finger_izz}"	-->
+<!--/> -->
+<link name="link_finger_1">
+        <visual>
+            <origin rpy="${M_PI/2-0.1} 0 ${M_PI/2}" xyz="-0.019 0 0" />
+            <geometry>
+                <mesh filename="package://phantomx_pincher/meshes/finger.dae"/>
+            </geometry>
+            <material name="Black"/>
+        </visual>
+        <inertial>
+            <mass value="${finger_mass}" />
+            <origin rpy="${M_PI/2} 0 ${M_PI/2}" xyz="0.006186000 0 0.011269000" />
+            <inertia ixx="${0}" ixy="${0}" ixz="${0}" iyy="${0}" iyz="${0}" izz="${0}" />
+        </inertial>
+        <collision>
+            <origin rpy="${M_PI/2-0.1} 0 ${M_PI/2}" xyz="-0.019 0 0" />
+            <geometry>
+                <mesh filename="package://phantomx_pincher/meshes/finger.dae"/>
+            </geometry>
+        </collision>
+    </link>
+ <link name="link_finger_2">
+        <visual>
+            <origin rpy="${M_PI/2-0.1} 0 ${M_PI/2}" xyz="-0.019 0 0" />
+            <geometry>
+                <mesh filename="package://phantomx_pincher/meshes/finger.dae"/>
+            </geometry>
+            <material name="Black"/>
+        </visual>
+        <inertial>
+            <mass value="${finger_mass}" />
+            <origin rpy="${M_PI/2} 0 ${M_PI/2}" xyz="0.006186000 0 0.011269000" />
+            <inertia ixx="${0}" ixy="${0}" ixz="${0}" iyy="${0}" iyz="${0}" izz="${0}" />
+        </inertial>
+        <collision>
+            <origin rpy="${M_PI/2-0.1} 0 ${M_PI/2}" xyz="-0.019 0 0" />
+            <geometry>
+                <mesh filename="package://phantomx_pincher/meshes/finger.dae"/>
+            </geometry>
+        </collision>
+    </link>
 <!-- Joint-Gripper-Camera-->
 <joint_camera
@@ -171,6 +211,6 @@
     parent="link_4"
     child="link_gripper_camera"
-    origin_rpy="0 0 0"
-    origin_xyz="${l4-0.015} 0 0"
+    origin_rpy="${M_PI/2} 0 ${M_PI/6}"
+    origin_xyz="${l4-0.02} -0.02 0"
     axis_xyz="0 0 1"
 />
@@ -179,4 +219,25 @@
     name="link_gripper_camera"
     origin_rpy="${M_PI/2} 0 0"
+    origin_xyz="0 0 0"
+    inertial_rpy="0 0 0"
+    inertial_xyz="${camera_size/2} 0 0"
+    mass="0"
+    ixx="0" ixy="0" ixz="0"
+    iyy="0" iyz="0" izz="0"
+/>
+<!-- Joint-Fixed-Camera-->
+<joint_camera
+    name="joint_camera_1"
+    type="fixed"
+    parent="world"
+    child="link_fixed_camera"
+    origin_rpy="0 -${M_PI/8} ${M_PI}"
+    origin_xyz="0.4 0 0"
+    axis_xyz="1 0 0"
+/>
+<!-- Link-Fixed-Camera-->
+<link_camera
+    name="link_fixed_camera"
+    origin_rpy="0 0 0"
     origin_xyz="0 0 0"
     inertial_rpy="0 0 0"
@@ -186,25 +247,4 @@
     iyy="${camera_iyy}" iyz="${camera_iyz}" izz="${camera_izz}"
 />
-<!-- Joint-Fixed-Camera-->
-<!--<joint_camera-->
-<!--    name="joint_camera_1" -->
-<!--    type="fixed"-->
-<!--    parent="world"-->
-<!--    child="link_fixed_camera"-->
-<!--    origin_rpy="0 0 ${8*M_PI/6}" -->
-<!--    origin_xyz="0.4 0.4 0"-->
-<!--    axis_xyz="1 0 0" -->
-<!--/>-->
-<!-- Link-Fixed-Camera-->
-<!--<link_camera-->
-<!--    name="link_fixed_camera"-->
-<!--    origin_rpy="0 0 0" -->
-<!--    origin_xyz="0 0 0"-->
-<!--    inertial_rpy="0 0 0" -->
-<!--    inertial_xyz="${camera_size/2} 0 0"-->
-<!--    mass="${camera_mass}"-->
-<!--    ixx="${camera_ixx}" ixy="${camera_ixy}" ixz="${camera_ixz}"-->
-<!--    iyy="${camera_iyy}" iyz="${camera_iyz}" izz="${camera_izz}"-->
-<!--/> -->
 <!-- -|-|-|-|-|-|-|-|- GAZEBO PLUGIN -|-|-|-|-|-|-|-|- -->
 <gazebo>
@@ -217,12 +257,12 @@
            <palm_link>link_4</palm_link>
            <gripper_link>link_finger_1</gripper_link>
-           <gripper_link>link_finger_1</gripper_link>
+           <gripper_link>link_finger_2</gripper_link>
         </arm>
        <forces_angle_tolerance>100</forces_angle_tolerance>
-       <update_rate>100</update_rate>
-       <grip_count_threshold>5</grip_count_threshold>
-       <max_grip_count>10</max_grip_count>
-       <release_tolerance>0.005</release_tolerance>
-       <disable_collisions_on_attach>true</disable_collisions_on_attach>
+       <update_rate>20</update_rate>
+       <grip_count_threshold>20</grip_count_threshold>
+       <max_grip_count>40</max_grip_count>
+       <release_tolerance>0.003</release_tolerance>
+       <disable_collisions_on_attach>false</disable_collisions_on_attach>
        <contact_topic>__default_topic__</contact_topic>
     </plugin>
@@ -234,6 +274,6 @@
     <horizontal_fov>1.3962634</horizontal_fov>
     <image>
-      <width>800</width>
-      <height>800</height>
+      <width>250</width>
+      <height>250</height>
       <format>R8G8B8</format>
     </image>
@@ -264,39 +304,39 @@
 </sensor>
 </gazebo>
-<!--<gazebo reference="link_fixed_camera">-->
-<!--<sensor type="camera" name="camera_1">-->
-<!--  <update_rate>5</update_rate>-->
-<!--  <camera name="head">-->
-<!--    <horizontal_fov>1.3962634</horizontal_fov>-->
-<!--    <image>-->
-<!--      <width>800</width>-->
-<!--      <height>800</height>-->
-<!--      <format>R8G8B8</format>-->
-<!--    </image>-->
-<!--    <clip>-->
-<!--      <near>0.02</near>-->
-<!--      <far>300</far>-->
-<!--    </clip>-->
-<!--    <noise>-->
-<!--      <type>gaussian</type>-->
-<!--      <mean>0.0</mean>-->
-<!--      <stddev>0.007</stddev>-->
-<!--    </noise>-->
-<!--  </camera>-->
-<!--  <plugin name="camera_controller" filename="libgazebo_ros_camera.so">-->
-<!--    <alwaysOn>true</alwaysOn>-->
-<!--    <updateRate>0.0</updateRate>-->
-<!--    <cameraName>camera_1</cameraName>-->
-<!--    <imageTopicName>image_raw</imageTopicName>-->
-<!--    <cameraInfoTopicName>camera_info</cameraInfoTopicName>-->
-<!--    <frameName>camera_link</frameName>-->
-<!--    <hackBaseline>0.07</hackBaseline>-->
-<!--    <distortionK1>0.0</distortionK1>-->
-<!--    <distortionK2>0.0</distortionK2>-->
-<!--    <distortionK3>0.0</distortionK3>-->
-<!--    <distortionT1>0.0</distortionT1>-->
-<!--    <distortionT2>0.0</distortionT2>-->
-<!--  </plugin>-->
-<!--</sensor>-->
-<!--</gazebo>-->
+<gazebo reference="link_fixed_camera">
+<sensor type="camera" name="camera_1">
+  <update_rate>5</update_rate>
+  <camera name="head">
+    <horizontal_fov>1.3962634</horizontal_fov>
+    <image>
+      <width>250</width>
+      <height>250</height>
+      <format>R8G8B8</format>
+    </image>
+    <clip>
+      <near>0.02</near>
+      <far>300</far>
+    </clip>
+    <noise>
+      <type>gaussian</type>
+      <mean>0.0</mean>
+      <stddev>0.007</stddev>
+    </noise>
+  </camera>
+  <plugin name="camera_controller" filename="libgazebo_ros_camera.so">
+    <alwaysOn>true</alwaysOn>
+    <updateRate>0.0</updateRate>
+    <cameraName>camera_1</cameraName>
+    <imageTopicName>image_raw</imageTopicName>
+    <cameraInfoTopicName>camera_info</cameraInfoTopicName>
+    <frameName>camera_link</frameName>
+    <hackBaseline>0.07</hackBaseline>
+    <distortionK1>0.0</distortionK1>
+    <distortionK2>0.0</distortionK2>
+    <distortionK3>0.0</distortionK3>
+    <distortionT1>0.0</distortionT1>
+    <distortionT2>0.0</distortionT2>
+  </plugin>
+</sensor>
+</gazebo>
 </robot>

File: Packages/phantomx_pincher/urdf/phantomx_description_inercias.xacro (robot description, xacro)
@@ -212,19 +212,19 @@
         <robotNamespace>/phantomx_pincher</robotNamespace>
     </plugin>
-<!--    <plugin name="gazebo_grasp_fix" filename="libgazebo_grasp_fix.so">-->
-<!--        <arm>-->
-<!--           <arm_name>phantomx_pincher</arm_name>-->
-<!--           <palm_link>link_4</palm_link>-->
-<!--           <gripper_link>link_finger_1</gripper_link>-->
-<!--           <gripper_link>link_finger_1</gripper_link>-->
-<!--        </arm>-->
-<!--       <forces_angle_tolerance>100</forces_angle_tolerance>-->
-<!--       <update_rate>5</update_rate>-->
-<!--       <grip_count_threshold>4</grip_count_threshold>-->
-<!--       <max_grip_count>8</max_grip_count>-->
-<!--       <release_tolerance>0.005</release_tolerance>-->
-<!--       <disable_collisions_on_attach>false</disable_collisions_on_attach>-->
-<!--       <contact_topic>__default_topic__</contact_topic>-->
-<!--    </plugin>-->
+    <plugin name="gazebo_grasp_fix" filename="libgazebo_grasp_fix.so">
+        <arm>
+           <arm_name>arm_pincher</arm_name>
+           <palm_link>link_4</palm_link>
+           <gripper_link>link_finger_1</gripper_link>
+           <gripper_link>link_finger_2</gripper_link>
+        </arm>
+       <forces_angle_tolerance>100</forces_angle_tolerance>
+       <update_rate>50</update_rate>
+       <grip_count_threshold>5</grip_count_threshold>
+       <max_grip_count>10</max_grip_count>
+       <release_tolerance>0.005</release_tolerance>
+       <disable_collisions_on_attach>false</disable_collisions_on_attach>
+       <contact_topic>__default_topic__</contact_topic>
+    </plugin>
 </gazebo>
 <gazebo reference="link_gripper_camera">

File: Packages/phantomx_pincher/urdf/phantomx_parameters.xacro (robot description, xacro)
@@ -8,5 +8,5 @@
 <xacro:property name="l3" value="0.107" />
 <xacro:property name="l4" value="0.0905" /> <!-- Agarre efectivo Gripper  -->
-<xacro:property name="offset_finger" value="0.03" />
+<xacro:property name="offset_finger" value="0.035" />
 <!-- Size of square 'camera' box -->
 <xacro:property name="camera_size" value="0.005" />
@@ -18,5 +18,47 @@
 </material>
 <!-- Mass and Inertia -->
-<xacro:property name="link_base_mass" value="0.33520"/>
+<!--<xacro:property name="link_base_mass" value="0.33520"/>-->
+<!--<xacro:property name="link_base_ixx" value="0.0"/>-->
+<!--<xacro:property name="link_base_ixy" value="0.0"/>-->
+<!--<xacro:property name="link_base_ixz" value="0.0"/>-->
+<!--<xacro:property name="link_base_iyy" value="0.0"/>-->
+<!--<xacro:property name="link_base_iyz" value="0.0"/>-->
+<!--<xacro:property name="link_base_izz" value="0.0"/>-->
+<!--<xacro:property name="link_1_mass" value="0.11748"/>-->
+<!--<xacro:property name="link_1_ixx" value="0.0"/>-->
+<!--<xacro:property name="link_1_ixy" value="0.0"/>-->
+<!--<xacro:property name="link_1_ixz" value="0.0"/>-->
+<!--<xacro:property name="link_1_iyy" value="0.0"/>-->
+<!--<xacro:property name="link_1_iyz" value="0.0"/>-->
+<!--<xacro:property name="link_1_izz" value="0.0"/>-->
+<!--<xacro:property name="link_2_mass" value="0.16239"/>-->
+<!--<xacro:property name="link_2_ixx" value="0.0"/>-->
+<!--<xacro:property name="link_2_ixy" value="0.0"/>-->
+<!--<xacro:property name="link_2_ixz" value="0.0"/>-->
+<!--<xacro:property name="link_2_iyy" value="0.0"/>-->
+<!--<xacro:property name="link_2_iyz" value="0.0"/>-->
+<!--<xacro:property name="link_2_izz" value="0.0"/>-->
+<!--<xacro:property name="link_3_mass" value="0.16239"/>-->
+<!--<xacro:property name="link_3_ixx" value="0.0"/>-->
+<!--<xacro:property name="link_3_ixy" value="0.0"/>-->
+<!--<xacro:property name="link_3_ixz" value="0.0"/>-->
+<!--<xacro:property name="link_3_iyy" value="0.0"/>-->
+<!--<xacro:property name="link_3_iyz" value="0.0"/>-->
+<!--<xacro:property name="link_3_izz" value="0.0"/>-->
+<!--<xacro:property name="link_4_mass" value="0.16012"/>-->
+<!--<xacro:property name="link_4_ixx" value="0.0"/>-->
+<!--<xacro:property name="link_4_ixy" value="0.0"/>-->
+<!--<xacro:property name="link_4_ixz" value="0.0"/>-->
+<!--<xacro:property name="link_4_iyy" value="0.0"/>-->
+<!--<xacro:property name="link_4_iyz" value="0.0"/>-->
+<!--<xacro:property name="link_4_izz" value="0.0"/>-->
+<!--<xacro:property name="finger_mass" value="0.01769"/>-->
+<!--<xacro:property name="finger_ixx" value="0.0"/>-->
+<!--<xacro:property name="finger_ixy" value="0.0"/>-->
+<!--<xacro:property name="finger_ixz" value="0.0"/>-->
+<!--<xacro:property name="finger_iyy" value="0.0"/>-->
+<!--<xacro:property name="finger_iyz" value="0.0"/>-->
+<!--<xacro:property name="finger_izz" value="0.0"/>-->
+<xacro:property name="link_base_mass" value="0.055"/>
 <xacro:property name="link_base_ixx" value="0.0"/>
 <xacro:property name="link_base_ixy" value="0.0"/>
@@ -25,5 +67,5 @@
 <xacro:property name="link_base_iyz" value="0.0"/>
 <xacro:property name="link_base_izz" value="0.0"/>
-<xacro:property name="link_1_mass" value="0.11748"/>
+<xacro:property name="link_1_mass" value="0.055"/>
 <xacro:property name="link_1_ixx" value="0.0"/>
 <xacro:property name="link_1_ixy" value="0.0"/>
@@ -32,5 +74,5 @@
 <xacro:property name="link_1_iyz" value="0.0"/>
 <xacro:property name="link_1_izz" value="0.0"/>
-<xacro:property name="link_2_mass" value="0.16239"/>
+<xacro:property name="link_2_mass" value="0.055"/>
 <xacro:property name="link_2_ixx" value="0.0"/>
 <xacro:property name="link_2_ixy" value="0.0"/>
@@ -39,5 +81,5 @@
 <xacro:property name="link_2_iyz" value="0.0"/>
 <xacro:property name="link_2_izz" value="0.0"/>
-<xacro:property name="link_3_mass" value="0.16239"/>
+<xacro:property name="link_3_mass" value="0.055"/>
 <xacro:property name="link_3_ixx" value="0.0"/>
 <xacro:property name="link_3_ixy" value="0.0"/>
@@ -46,5 +88,5 @@
 <xacro:property name="link_3_iyz" value="0.0"/>
 <xacro:property name="link_3_izz" value="0.0"/>
-<xacro:property name="link_4_mass" value="0.16012"/>
+<xacro:property name="link_4_mass" value="0.055"/>
 <xacro:property name="link_4_ixx" value="0.0"/>
 <xacro:property name="link_4_ixy" value="0.0"/>
@@ -53,11 +95,11 @@
 <xacro:property name="link_4_iyz" value="0.0"/>
 <xacro:property name="link_4_izz" value="0.0"/>
-<xacro:property name="finger_mass" value="0.01769"/>
-<xacro:property name="finger_ixx" value="0.0"/>
-<xacro:property name="finger_ixy" value="0.0"/>
-<xacro:property name="finger_ixz" value="0.0"/>
-<xacro:property name="finger_iyy" value="0.0"/>
-<xacro:property name="finger_iyz" value="0.0"/>
-<xacro:property name="finger_izz" value="0.0"/>
+<xacro:property name="finger_mass" value="0.006803850"/>
+<xacro:property name="finger_ixx" value="0.000001127"/>
+<xacro:property name="finger_ixy" value="0.000000000"/>
+<xacro:property name="finger_ixz" value="0.000000000"/>
+<xacro:property name="finger_iyy" value="0.000001776"/>
+<xacro:property name="finger_iyz" value="-0.000000278"/>
+<xacro:property name="finger_izz" value="0.000001162"/>
 <!-- Joint-Servomotor Position Limits -150,150 deg -->
 <xacro:property name="joint_lower" value="-2.61799" />
@@ -170,10 +212,10 @@
                 <box size="${camera_size} ${camera_size} ${camera_size}"/>
             </geometry>
-            <material name="red"/>
+            <material name="Black"/>
         </visual>
         <inertial>
-            <mass value="0" />
+            <mass value="${mass}" />
             <origin rpy="${inertial_rpy}" xyz="${inertial_xyz}" />
-            <inertia ixx="0" ixy="0" ixz="0" iyy="0" iyz="0" izz="0" />
+            <inertia ixx="${ixx}" ixy="${ixy}" ixz="${ixz}" iyy="${iyy}" iyz="${iyz}" izz="${izz}" />
         </inertial>
     </link>

File: Packages/phantomx_pincher/urdf/rosca_description.xacro (robot description, xacro)
@@ -9,5 +9,5 @@
         <origin rpy="0 0 0" xyz="0 0 0" />
         <geometry>
-            <mesh filename="package://phantomx_pincher/meshes/rosca.stl" scale="${M_SCALE} ${M_SCALE} ${M_SCALE}"/>
+            <mesh filename="package://phantomx_pincher/meshes/rosca.stl" scale="${M_SCALE} ${M_SCALE} 0.013"/>
         </geometry>
     </visual>
@@ -20,5 +20,5 @@
         <origin rpy="0 0 0" xyz="0 0 0" />
         <geometry>
-            <mesh filename="package://phantomx_pincher/meshes/rosca.stl" scale="${M_SCALE} ${M_SCALE} ${M_SCALE}"/>
+            <mesh filename="package://phantomx_pincher/meshes/rosca.stl" scale="${M_SCALE} ${M_SCALE} 0.013"/>
         </geometry>
     </collision>
